Commit message: fix:修复配置

File: src/robot_description/urdf/mobile_manipulator.urdf.xacro (robot description, xacro)
@@ -470,3 +470,40 @@
   </gazebo>
   </xacro:if>
+  <!-- ============================ ros2_control ============================= -->
+  <!-- 这一块**不是**给 Gazebo 看的，是给 ros2_control 看的：它声明"这台机器有哪几个
+       关节、各暴露什么接口、由哪个硬件插件驱动"。
+       ⚠️ 用 `mock_components/GenericSystem` 当硬件 —— 它是 ros2_control 自带的**假硬件**：
+          写进 command_interface 的值直接出现在 state_interface 上（`calculate_dynamics`
+          默认 false ⇒ 命令即状态）。于是**不需要 Gazebo、不需要真机**，
+          整条 ros2_control 栈（controller_manager → joint_trajectory_controller）就能跑。
+          要换成真机，只改 `<plugin>` 那一行。
+       ⚠️ Gazebo 那一段（下面的 <gazebo> 标签）和这一块是**两套独立的方案**，
+          互不打扰：前者靠 gz-sim 的插件，后者靠 ros2_control。
+       ⚠️ 只声明确实要控的 5 个关节（4 个手臂 + 1 个夹爪）。
+          车轮是 continuous 且没人控它们，混进来只会让 /joint_states 多出两条无意义的 0。 -->
+  <ros2_control name="mobile_manipulator" type="system">
+    <hardware>
+      <plugin>mock_components/GenericSystem</plugin>
+    </hardware>
+    <joint name="shoulder_pan_joint">
+      <command_interface name="position"/>
+      <state_interface name="position"/>
+    </joint>
+    <joint name="shoulder_lift_joint">
+      <command_interface name="position"/>
+      <state_interface name="position"/>
+    </joint>
+    <joint name="elbow_joint">
+      <command_interface name="position"/>
+      <state_interface name="position"/>
+    </joint>
+    <joint name="wrist_joint">
+      <command_interface name="position"/>
+      <state_interface name="position"/>
+    </joint>
+    <joint name="gripper_joint">
+      <command_interface name="position"/>
+      <state_interface name="position"/>
+    </joint>
+  </ros2_control>
 </robot>

Commit message: fix:修复配置&&简化注释

File: src/robot_description/urdf/mobile_manipulator.urdf.xacro (robot description, xacro)
@@ -18,4 +18,9 @@
   <xacro:property name="forearm_length" value="0.20"/>
   <xacro:property name="wrist_length" value="0.06"/>
+  <!-- 腕部后两个自由度各占一小段。加它们是为了把 arm 凑够 **6 个 revolute**：
+       只有 4 个的时候 KDL 解不出 6 维位姿（欠自由度），只能靠 position_only_ik
+       放弃姿态、只保位置。 -->
+  <xacro:property name="wrist_pitch_length" value="0.03"/>
+  <xacro:property name="wrist_roll_length" value="0.02"/>
   <xacro:property name="arm_radius" value="0.035"/>
   <!-- ================================ Inertia =============================== -->
@@ -295,4 +300,61 @@
     <dynamics damping="0.1" friction="0.0"/>
   </joint>
+  <!-- 腕部第 2、3 段：Z-Y-Z 球形腕，和 pan/lift/elbow 一起构成 6R。
+       ⚠️ 第 3 段轴必须是 Z：夹爪沿 +Z 装在这个法兰上，绕工具轴自转就是绕 Z。
+       ⚠️ pitch = 0 时第 1、3 段共线，是 Z-Y-Z 固有的奇异位形，不是建模错误。 -->
+  <link name="wrist_pitch_link">
+    <visual>
+      <origin xyz="0 0 ${wrist_pitch_length / 2.0}" rpy="0 0 0"/>
+      <geometry>
+        <cylinder radius="${arm_radius * 0.7}" length="${wrist_pitch_length}"/>
+      </geometry>
+      <material name="orange">
+        <color rgba="0.9 0.45 0.1 1.0"/>
+      </material>
+    </visual>
+    <collision>
+      <origin xyz="0 0 ${wrist_pitch_length / 2.0}" rpy="0 0 0"/>
+      <geometry>
+        <cylinder radius="${arm_radius * 0.7}" length="${wrist_pitch_length}"/>
+      </geometry>
+    </collision>
+    <xacro:cylinder_inertial mass="0.2" radius="${arm_radius * 0.7}"
+                              length="${wrist_pitch_length}"/>
+  </link>
+  <joint name="wrist_pitch_joint" type="revolute">
+    <parent link="wrist_link"/>
+    <child link="wrist_pitch_link"/>
+    <origin xyz="0 0 ${wrist_length}" rpy="0 0 0"/>
+    <axis xyz="0 1 0"/>
+    <limit lower="-1.6" upper="1.6" effort="10.0" velocity="2.0"/>
+    <dynamics damping="0.1" friction="0.0"/>
+  </joint>
+  <link name="wrist_roll_link">
+    <visual>
+      <origin xyz="0 0 ${wrist_roll_length / 2.0}" rpy="0 0 0"/>
+      <geometry>
+        <cylinder radius="${arm_radius * 0.6}" length="${wrist_roll_length}"/>
+      </geometry>
+      <material name="grey">
+        <color rgba="0.35 0.37 0.40 1.0"/>
+      </material>
+    </visual>
+    <collision>
+      <origin xyz="0 0 ${wrist_roll_length / 2.0}" rpy="0 0 0"/>
+      <geometry>
+        <cylinder radius="${arm_radius * 0.6}" length="${wrist_roll_length}"/>
+      </geometry>
+    </collision>
+    <xacro:cylinder_inertial mass="0.15" radius="${arm_radius * 0.6}"
+                              length="${wrist_roll_length}"/>
+  </link>
+  <joint name="wrist_roll_joint" type="revolute">
+    <parent link="wrist_pitch_link"/>
+    <child link="wrist_roll_link"/>
+    <origin xyz="0 0 ${wrist_pitch_length}" rpy="0 0 0"/>
+    <axis xyz="0 0 1"/>
+    <limit lower="-3.14" upper="3.14" effort="5.0" velocity="2.0"/>
+    <dynamics damping="0.05" friction="0.0"/>
+  </joint>
   <!-- ============================== Gripper ================================ -->
   <link name="gripper_base_link">
@@ -313,7 +375,7 @@
   </link>
   <joint name="gripper_base_joint" type="fixed">
-    <parent link="wrist_link"/>
+    <parent link="wrist_roll_link"/>
     <child link="gripper_base_link"/>
-    <origin xyz="0 0 ${wrist_length + 0.01}" rpy="0 0 0"/>
+    <origin xyz="0 0 ${wrist_roll_length + 0.01}" rpy="0 0 0"/>
   </joint>
   <xacro:macro name="finger" params="prefix y">
@@ -391,4 +453,6 @@
       <joint_name>elbow_joint</joint_name>
       <joint_name>wrist_joint</joint_name>
+      <joint_name>wrist_pitch_joint</joint_name>
+      <joint_name>wrist_roll_joint</joint_name>
       <joint_name>gripper_joint</joint_name>
     </plugin>
@@ -407,4 +471,6 @@
   <xacro:arm_position_controller joint="elbow_joint"/>
   <xacro:arm_position_controller joint="wrist_joint"/>
+  <xacro:arm_position_controller joint="wrist_pitch_joint"/>
+  <xacro:arm_position_controller joint="wrist_roll_joint"/>
   <xacro:arm_position_controller joint="gripper_joint"/>
   <gazebo reference="laser_link">
@@ -471,15 +537,6 @@
   </xacro:if>
   <!-- ============================ ros2_control ============================= -->
-  <!-- 这一块**不是**给 Gazebo 看的，是给 ros2_control 看的：它声明"这台机器有哪几个
-       关节、各暴露什么接口、由哪个硬件插件驱动"。
-       ⚠️ 用 `mock_components/GenericSystem` 当硬件 —— 它是 ros2_control 自带的**假硬件**：
-          写进 command_interface 的值直接出现在 state_interface 上（`calculate_dynamics`
-          默认 false ⇒ 命令即状态）。于是**不需要 Gazebo、不需要真机**，
-          整条 ros2_control 栈（controller_manager → joint_trajectory_controller）就能跑。
-          要换成真机，只改 `<plugin>` 那一行。
-       ⚠️ Gazebo 那一段（下面的 <gazebo> 标签）和这一块是**两套独立的方案**，
-          互不打扰：前者靠 gz-sim 的插件，后者靠 ros2_control。
-       ⚠️ 只声明确实要控的 5 个关节（4 个手臂 + 1 个夹爪）。
-          车轮是 continuous 且没人控它们，混进来只会让 /joint_states 多出两条无意义的 0。 -->
+  <!-- 给 ros2_control 用的：声明关节、接口、硬件插件。用 mock_components/GenericSystem
+       假硬件（命令即状态，不需要 Gazebo）。只声明要控的 7 个关节，车轮没人控。 -->
   <ros2_control name="mobile_manipulator" type="system">
     <hardware>
@@ -502,4 +559,12 @@
       <state_interface name="position"/>
     </joint>
+    <joint name="wrist_pitch_joint">
+      <command_interface name="position"/>
+      <state_interface name="position"/>
+    </joint>
+    <joint name="wrist_roll_joint">
+      <command_interface name="position"/>
+      <state_interface name="position"/>
+    </joint>
     <joint name="gripper_joint">
       <command_interface name="position"/>

Commit message: feat:接入UR5实模并修复RViz可视化
- arm 换官方 UR5 模型（真实运动学与网格），保留原 link/joint 名
- 加 0.5m 底座避免零位自碰；SRDF 补底座 disable_collisions
- mock 发布 /robot_description、补轮子 TF；launch 起 robot_state_publisher
- RViz 打开 RobotModel、描述用瞬态 local、合并重复 black 材质
- 探针关节限位改从 URDF 读；真实栈 fixture 先回零位

File: src/robot_description/urdf/mobile_manipulator.urdf.xacro (robot description, xacro)
@@ -21,13 +21,7 @@
   <xacro:property name="wheel_offset_x" value="0.13"/>
   <xacro:property name="wheel_offset_y" value="0.185"/>
-  <xacro:property name="arm_base_height" value="0.06"/>
-  <xacro:property name="upper_arm_length" value="0.22"/>
-  <xacro:property name="forearm_length" value="0.20"/>
-  <xacro:property name="wrist_length" value="0.06"/>
   <!-- 腕部后两个自由度各占一小段。arm 组靠它们凑够 **6 个 revolute** ——
        KDL 才能解完整 6 维位姿（少一个就退化成欠自由度，解不出带姿态的目标）。 -->
-  <xacro:property name="wrist_pitch_length" value="0.03"/>
   <xacro:property name="wrist_roll_length" value="0.02"/>
-  <xacro:property name="arm_radius" value="0.035"/>
   <!-- ================================ Inertia =============================== -->
   <xacro:macro name="box_inertial" params="mass x y z">
@@ -62,5 +56,5 @@
       </geometry>
       <material name="grey">
-        <color rgba="0.35 0.37 0.40 1.0"/>
+        <color rgba="0.10 0.20 0.45 1.0"/>
       </material>
     </visual>
@@ -183,185 +177,211 @@
   </joint>
   <!-- =============================== Arm =================================== -->
+  <!-- ═══ 手臂：官方 UR5 ═══════════════════════════════════════════════
+       为什么是"照抄"而不是自己捏：mesh 本身就是按 UR5 的**真实尺寸**做的，
+       几何与 mesh 不一致时模型会在关节处断开。数值来源（本机已装，见 docs/visualization.md）：
+         ur_description/config/ur5/default_kinematics.yaml   ← 6 个关节的 xyz/rpy
+         ur_description/config/ur5/joint_limits.yaml          ← 限位/速度/力矩（已换算成弧度）
+         ur_description/config/ur5/visual_parameters.yaml     ← 每个 link 用哪个 mesh、视觉偏移
+       ⚠️ 名字仍用**我们自己的**（wrist / wrist_pitch / wrist_roll ↔ UR 的 wrist_1/2/3）：
+          这样 SRDF、MoveIt 配置、mock、测试都不用跟着改。 -->
   <link name="arm_base_link">
     <visual>
-      <geometry>
-        <cylinder radius="0.055" length="${arm_base_height}"/>
-      </geometry>
-      <material name="orange">
-        <color rgba="0.9 0.45 0.1 1.0"/>
-      </material>
-    </visual>
-    <collision>
-      <geometry>
-        <cylinder radius="0.055" length="${arm_base_height}"/>
-      </geometry>
-    </collision>
-    <xacro:cylinder_inertial mass="0.6" radius="0.055" length="${arm_base_height}"/>
-  </link>
+      <origin xyz="0 0 0" rpy="0 0 ${PI}"/>
+      <geometry>
+        <mesh filename="package://ur_description/meshes/ur5/visual/base.dae"/>
+      </geometry>
+      <material name="ur_light_grey">
+        <color rgba="0.7 0.7 0.7 1.0"/>
+      </material>
+    </visual>
+    <collision>
+      <origin xyz="0 0 0" rpy="0 0 ${PI}"/>
+      <geometry>
+        <mesh filename="package://ur_description/meshes/ur5/collision/base.stl"/>
+      </geometry>
+    </collision>
+    <xacro:cylinder_inertial mass="4.0" radius="0.06" length="0.06"/>
+  </link>
+  <!-- 手臂基座：UR5 在零位是**横躺**的，直接装在底盘顶面必然穿模
+       （MoveIt 的碰撞检查当场就会把零位判成自碰撞）。真实移动机械臂都这么抬一段。 -->
+  <link name="arm_pedestal_link">
+    <visual>
+      <origin xyz="0 0 0.25" rpy="0 0 0"/>
+      <geometry>
+        <cylinder radius="0.05" length="0.50"/>
+      </geometry>
+      <material name="dark_grey">
+        <color rgba="0.25 0.27 0.30 1.0"/>
+      </material>
+    </visual>
+    <collision>
+      <origin xyz="0 0 0.25" rpy="0 0 0"/>
+      <geometry>
+        <cylinder radius="0.05" length="0.50"/>
+      </geometry>
+    </collision>
+    <xacro:cylinder_inertial mass="2.2" radius="0.05" length="0.50"/>
+  </link>
+  <joint name="arm_pedestal_joint" type="fixed">
+    <parent link="base_link"/>
+    <child link="arm_pedestal_link"/>
+    <origin xyz="0 0 ${base_height / 2.0}" rpy="0 0 0"/>
+  </joint>
   <joint name="arm_base_joint" type="fixed">
-    <parent link="base_link"/>
+    <parent link="arm_pedestal_link"/>
     <child link="arm_base_link"/>
-    <origin xyz="-0.05 0 ${base_height / 2.0 + arm_base_height / 2.0}" rpy="0 0 0"/>
+    <origin xyz="0 0 0.50" rpy="0 0 0"/>
   </joint>
   <link name="shoulder_link">
     <visual>
-      <geometry>
-        <cylinder radius="${arm_radius}" length="0.06"/>
-      </geometry>
-      <material name="orange">
-        <color rgba="0.9 0.45 0.1 1.0"/>
-      </material>
-    </visual>
-    <collision>
-      <geometry>
-        <cylinder radius="${arm_radius}" length="0.06"/>
-      </geometry>
-    </collision>
-    <xacro:cylinder_inertial mass="0.4" radius="${arm_radius}" length="0.06"/>
+      <origin xyz="0 0 0" rpy="0 0 ${PI}"/>
+      <geometry>
+        <mesh filename="package://ur_description/meshes/ur5/visual/shoulder.dae"/>
+      </geometry>
+      <material name="ur_light_grey">
+        <color rgba="0.7 0.7 0.7 1.0"/>
+      </material>
+    </visual>
+    <collision>
+      <origin xyz="0 0 0" rpy="0 0 ${PI}"/>
+      <geometry>
+        <mesh filename="package://ur_description/meshes/ur5/collision/shoulder.stl"/>
+      </geometry>
+    </collision>
+    <xacro:cylinder_inertial mass="3.7" radius="0.06" length="0.12"/>
   </link>
   <joint name="shoulder_pan_joint" type="revolute">
     <parent link="arm_base_link"/>
     <child link="shoulder_link"/>
-    <origin xyz="0 0 ${arm_base_height / 2.0 + 0.03}" rpy="0 0 0"/>
+    <origin xyz="0 0 0.089159" rpy="0 0 0"/>
     <axis xyz="0 0 1"/>
-    <limit lower="-3.14" upper="3.14" effort="30.0" velocity="2.0"/>
-    <dynamics damping="0.1" friction="0.0"/>
+    <limit lower="-6.283185307" upper="6.283185307" effort="150.0" velocity="3.14159265"/>
   </joint>
   <link name="upper_arm_link">
     <visual>
-      <origin xyz="0 0 ${upper_arm_length / 2.0}" rpy="0 0 0"/>
-      <geometry>
-        <cylinder radius="${arm_radius}" length="${upper_arm_length}"/>
-      </geometry>
-      <material name="orange">
-        <color rgba="0.9 0.45 0.1 1.0"/>
-      </material>
-    </visual>
-    <collision>
-      <origin xyz="0 0 ${upper_arm_length / 2.0}" rpy="0 0 0"/>
-      <geometry>
-        <cylinder radius="${arm_radius}" length="${upper_arm_length}"/>
-      </geometry>
-    </collision>
-    <xacro:cylinder_inertial mass="0.9" radius="${arm_radius}" length="${upper_arm_length}"/>
+      <origin xyz="0 0 0.13585" rpy="${PI / 2.0} 0 ${-PI / 2.0}"/>
+      <geometry>
+        <mesh filename="package://ur_description/meshes/ur5/visual/upperarm.dae"/>
+      </geometry>
+      <material name="ur_light_grey">
+        <color rgba="0.7 0.7 0.7 1.0"/>
+      </material>
+    </visual>
+    <collision>
+      <origin xyz="0 0 0.13585" rpy="${PI / 2.0} 0 ${-PI / 2.0}"/>
+      <geometry>
+        <mesh filename="package://ur_description/meshes/ur5/collision/upperarm.stl"/>
+      </geometry>
+    </collision>
+    <xacro:cylinder_inertial mass="8.393" radius="0.054" length="0.4"/>
   </link>
   <joint name="shoulder_lift_joint" type="revolute">
     <parent link="shoulder_link"/>
     <child link="upper_arm_link"/>
-    <origin xyz="0 0 0.03" rpy="0 0 0"/>
-    <axis xyz="0 1 0"/>
-    <limit lower="-1.8" upper="1.8" effort="30.0" velocity="2.0"/>
-    <dynamics damping="0.1" friction="0.0"/>
+    <origin xyz="0 0 0" rpy="${PI / 2.0} 0 0"/>
+    <axis xyz="0 0 1"/>
+    <limit lower="-6.283185307" upper="6.283185307" effort="150.0" velocity="3.14159265"/>
   </joint>
   <link name="forearm_link">
     <visual>
-      <origin xyz="0 0 ${forearm_length / 2.0}" rpy="0 0 0"/>
-      <geometry>
-        <cylinder radius="${arm_radius * 0.9}" length="${forearm_length}"/>
-      </geometry>
-      <material name="orange">
-        <color rgba="0.9 0.45 0.1 1.0"/>
-      </material>
-    </visual>
-    <collision>
-      <origin xyz="0 0 ${forearm_length / 2.0}" rpy="0 0 0"/>
-      <geometry>
-        <cylinder radius="${arm_radius * 0.9}" length="${forearm_length}"/>
-      </geometry>
-    </collision>
-    <xacro:cylinder_inertial mass="0.7" radius="${arm_radius * 0.9}" length="${forearm_length}"/>
+      <origin xyz="0 0 0.0165" rpy="${PI / 2.0} 0 ${-PI / 2.0}"/>
+      <geometry>
+        <mesh filename="package://ur_description/meshes/ur5/visual/forearm.dae"/>
+      </geometry>
+      <material name="ur_light_grey">
+        <color rgba="0.7 0.7 0.7 1.0"/>
+      </material>
+    </visual>
+    <collision>
+      <origin xyz="0 0 0.0165" rpy="${PI / 2.0} 0 ${-PI / 2.0}"/>
+      <geometry>
+        <mesh filename="package://ur_description/meshes/ur5/collision/forearm.stl"/>
+      </geometry>
+    </collision>
+    <xacro:cylinder_inertial mass="2.33" radius="0.04" length="0.39"/>
   </link>
   <joint name="elbow_joint" type="revolute">
     <parent link="upper_arm_link"/>
     <child link="forearm_link"/>
-    <origin xyz="0 0 ${upper_arm_length}" rpy="0 0 0"/>
-    <axis xyz="0 1 0"/>
-    <limit lower="-2.4" upper="2.4" effort="20.0" velocity="2.0"/>
-    <dynamics damping="0.1" friction="0.0"/>
+    <origin xyz="-0.425 0 0" rpy="0 0 0"/>
+    <axis xyz="0 0 1"/>
+    <!-- UR 官方把肘关节人为限制在 ±180°（超过之后肩部会挡住，规划空间会分裂） -->
+    <limit lower="-3.14159265" upper="3.14159265" effort="150.0" velocity="3.14159265"/>
   </joint>
   <link name="wrist_link">
     <visual>
-      <origin xyz="0 0 ${wrist_length / 2.0}" rpy="0 0 0"/>
-      <geometry>
-        <cylinder radius="${arm_radius * 0.8}" length="${wrist_length}"/>
-      </geometry>
-      <material name="orange">
-        <color rgba="0.9 0.45 0.1 1.0"/>
-      </material>
-    </visual>
-    <collision>
-      <origin xyz="0 0 ${wrist_length / 2.0}" rpy="0 0 0"/>
-      <geometry>
-        <cylinder radius="${arm_radius * 0.8}" length="${wrist_length}"/>
-      </geometry>
-    </collision>
-    <xacro:cylinder_inertial mass="0.3" radius="${arm_radius * 0.8}" length="${wrist_length}"/>
+      <origin xyz="0 0 -0.093" rpy="${PI / 2.0} 0 0"/>
+      <geometry>
+        <mesh filename="package://ur_description/meshes/ur5/visual/wrist1.dae"/>
+      </geometry>
+      <material name="ur_light_grey">
+        <color rgba="0.7 0.7 0.7 1.0"/>
+      </material>
+    </visual>
+    <collision>
+      <origin xyz="0 0 -0.093" rpy="${PI / 2.0} 0 0"/>
+      <geometry>
+        <mesh filename="package://ur_description/meshes/ur5/collision/wrist1.stl"/>
+      </geometry>
+    </collision>
+    <xacro:cylinder_inertial mass="1.219" radius="0.045" length="0.09"/>
   </link>
   <joint name="wrist_joint" type="revolute">
     <parent link="forearm_link"/>
     <child link="wrist_link"/>
-    <origin xyz="0 0 ${forearm_length}" rpy="0 0 0"/>
+    <origin xyz="-0.39225 0 0.10915" rpy="0 0 0"/>
     <axis xyz="0 0 1"/>
-    <limit lower="-3.14" upper="3.14" effort="10.0" velocity="2.0"/>
-    <dynamics damping="0.1" friction="0.0"/>
-  </joint>
-  <!-- 腕部第 2、3 段：Z-Y-Z 球形腕，和 pan/lift/elbow 一起构成 6R。
-       ⚠️ 第 3 段轴必须是 Z：夹爪沿 +Z 装在这个法兰上，绕工具轴自转就是绕 Z。
-       ⚠️ pitch = 0 时第 1、3 段共线，是 Z-Y-Z 固有的奇异位形，不是建模错误。 -->
+    <limit lower="-6.283185307" upper="6.283185307" effort="28.0" velocity="3.14159265"/>
+  </joint>
   <link name="wrist_pitch_link">
     <visual>
-      <origin xyz="0 0 ${wrist_pitch_length / 2.0}" rpy="0 0 0"/>
-      <geometry>
-        <cylinder radius="${arm_radius * 0.7}" length="${wrist_pitch_length}"/>
-      </geometry>
-      <material name="orange">
-        <color rgba="0.9 0.45 0.1 1.0"/>
-      </material>
-    </visual>
-    <collision>
-      <origin xyz="0 0 ${wrist_pitch_length / 2.0}" rpy="0 0 0"/>
-      <geometry>
-        <cylinder radius="${arm_radius * 0.7}" length="${wrist_pitch_length}"/>
-      </geometry>
-    </collision>
-    <xacro:cylinder_inertial mass="0.2" radius="${arm_radius * 0.7}"
-                              length="${wrist_pitch_length}"/>
+      <origin xyz="0 0 -0.095" rpy="0 0 0"/>
+      <geometry>
+        <mesh filename="package://ur_description/meshes/ur5/visual/wrist2.dae"/>
+      </geometry>
+      <material name="ur_light_grey">
+        <color rgba="0.7 0.7 0.7 1.0"/>
+      </material>
+    </visual>
+    <collision>
+      <origin xyz="0 0 -0.095" rpy="0 0 0"/>
+      <geometry>
+        <mesh filename="package://ur_description/meshes/ur5/collision/wrist2.stl"/>
+      </geometry>
+    </collision>
+    <xacro:cylinder_inertial mass="1.219" radius="0.045" length="0.09"/>
   </link>
   <joint name="wrist_pitch_joint" type="revolute">
     <parent link="wrist_link"/>
     <child link="wrist_pitch_link"/>
-    <origin xyz="0 0 ${wrist_length}" rpy="0 0 0"/>
-    <axis xyz="0 1 0"/>
-    <limit lower="-1.6" upper="1.6" effort="10.0" velocity="2.0"/>
-    <dynamics damping="0.1" friction="0.0"/>
+    <origin xyz="0 -0.09465 0" rpy="${PI / 2.0} 0 0"/>
+    <axis xyz="0 0 1"/>
+    <limit lower="-6.283185307" upper="6.283185307" effort="28.0" velocity="3.14159265"/>
   </joint>
   <link name="wrist_roll_link">
     <visual>
-      <origin xyz="0 0 ${wrist_roll_length / 2.0}" rpy="0 0 0"/>
-      <geometry>
-        <cylinder radius="${arm_radius * 0.6}" length="${wrist_roll_length}"/>
-      </geometry>
-      <material name="grey">
-        <color rgba="0.35 0.37 0.40 1.0"/>
-      </material>
-    </visual>
-    <collision>
-      <origin xyz="0 0 ${wrist_roll_length / 2.0}" rpy="0 0 0"/>
-      <geometry>
-        <cylinder radius="${arm_radius * 0.6}" length="${wrist_roll_length}"/>
-      </geometry>
-    </collision>
-    <xacro:cylinder_inertial mass="0.15" radius="${arm_radius * 0.6}"
-                              length="${wrist_roll_length}"/>
+      <origin xyz="0 0 -0.0818" rpy="${PI / 2.0} 0 0"/>
+      <geometry>
+        <mesh filename="package://ur_description/meshes/ur5/visual/wrist3.dae"/>
+      </geometry>
+      <material name="ur_light_grey">
+        <color rgba="0.7 0.7 0.7 1.0"/>
+      </material>
+    </visual>
+    <collision>
+      <origin xyz="0 0 -0.0818" rpy="${PI / 2.0} 0 0"/>
+      <geometry>
+        <mesh filename="package://ur_description/meshes/ur5/collision/wrist3.stl"/>
+      </geometry>
+    </collision>
+    <xacro:cylinder_inertial mass="0.1879" radius="0.045" length="0.08"/>
   </link>
   <joint name="wrist_roll_joint" type="revolute">
     <parent link="wrist_pitch_link"/>
     <child link="wrist_roll_link"/>
-    <origin xyz="0 0 ${wrist_pitch_length}" rpy="0 0 0"/>
+    <origin xyz="0 0.0823 0" rpy="${PI / 2.0} ${PI} ${PI}"/>
     <axis xyz="0 0 1"/>
-    <limit lower="-3.14" upper="3.14" effort="5.0" velocity="2.0"/>
-    <dynamics damping="0.05" friction="0.0"/>
-  </joint>
-  <!-- ============================== Gripper ================================ -->
+    <limit lower="-6.283185307" upper="6.283185307" effort="28.0" velocity="3.14159265"/>
+  </joint>
   <link name="gripper_base_link">
     <visual>
@@ -370,5 +390,5 @@
       </geometry>
       <material name="black">
-        <color rgba="0.1 0.1 0.1 1.0"/>
+        <color rgba="0.05 0.05 0.05 1.0"/>
       </material>
     </visual>
@@ -393,5 +413,5 @@
         </geometry>
         <material name="black">
-          <color rgba="0.1 0.1 0.1 1.0"/>
+          <color rgba="0.05 0.05 0.05 1.0"/>
         </material>
       </visual>
