Commit message: fix:传感器挂载帧统一到URDF（消除重复TF）
- mock 不再自己广播激光/IMU/相机的挂载 TF：它们是 URDF 的 fixed joint，按 ROS 约定归
  robot_state_publisher 发到 /tf_static（自己再发一份 = 同一帧两个父节点 ⇒ TF_REPEATED_DATA）
- mock 需要的挂载量（激光/相机的 x/z）改为从 URDF 读，不再抄数字；URDF 补 camera_optical_frame
- /scan 的 frame_id 由 laser_frame 改为 laser_link（破坏性：按帧名投影的消费方需同步）
- 抽出 mock_world.hpp（房间常量 + rayToBox 纯函数）并补单测；测试里 LyingNavigateServer 改名 FakeNavigateServer

File: src/robot_description/urdf/mobile_manipulator.urdf.xacro (robot description, xacro)
@@ -175,4 +175,13 @@
     <child link="camera_link"/>
     <origin xyz="${base_length / 2.0 - 0.01} 0 ${base_height / 2.0 + 0.05}" rpy="0 0 0"/>
+  </joint>
+  <!-- 光学帧：ROS 约定图像在 z 朝前 / x 朝右 / y 朝下的坐标系里，与 body 系差一个固定旋转。
+       ⚠️ 它必须由 URDF 提供（fixed joint ⇒ 由 robot_state_publisher 发到 /tf_static）：
+       少了它，消费方拿 TF 投影深度图会得到"错误但看起来合理"的结果。 -->
+  <link name="camera_optical_frame"/>
+  <joint name="camera_optical_joint" type="fixed">
+    <parent link="camera_link"/>
+    <child link="camera_optical_frame"/>
+    <origin xyz="0 0 0" rpy="-1.57079632679 0 -1.57079632679"/>
   </joint>
   <!-- =============================== Arm =================================== -->

Commit message: feat:底盘改由标准 diff_drive_controller 驱动（与手臂同一套 ros2_control）
原来底盘走 gz 私有的 DiffDrive 插件、手臂走 ros2_control —— 两套驱动机制。现在底盘也
纳入 ros2_control，整机只剩一套：接真机时换的是**同一个**硬件插件，接口不变。

改法（都是被 Jazzy 的事实逼出来的，不是自由选择）：
· diff_drive_controller **只收 TwistStamped**（实测 .so 里只有 TwistStamped 的符号，
  没有 use_stamped_vel 开关、也没有 unstamped 订阅）⇒ nav2 侧开
  enable_stamped_cmd_vel，mock 的 cmd_vel 订阅同步改成 stamped。
  ⚠️ cmd_vel 不属于 SDK 契约（见 docs/robot-flows.md）⇒ 不破契约。
· 控制器话题是 ~/cmd_vel、~/odom（节点名带控制器名 ⇒ /diff_drive_controller/cmd_vel）
  ⇒ 用 spawner 的 --controller-ros-args 重映射回 /cmd_vel、/odom，不插转换节点。
  controller_manager 自带的 --remap 官方已标废弃，提示里点名要改用这个参数。
· enable_odom_tf: false —— TF 仍由 odom_tf_broadcaster 独家发，避免两个作者改
  odom→base 让 TF 抖。车轮状态继续由 gz 的 JointStatePublisher 经桥发
  （joint_state_broadcaster 仍只列手臂），所以桥里没有多出重复发布者。
· 桥 9 条减到 7 条：删掉 /cmd_vel(ROS→GZ) 与 /odom(GZ→ROS) —— 两侧都在 ROS 侧了，
  留着只会多出"无人消费的 gz /cmd_vel"和两个 /odom 作者。

实测（headless Gazebo）：
· 三个控制器都 active，其中 diff_drive_controller 4 s 内起来
· 发 /cmd_vel = TwistStamped(linear.x=0.2) 持续 4 s ⇒ /odom 的 x：0 → 0.848
  （≈ 0.2 m/s × 4.2 s，y ≈ 0）⇒ 里程计真的在跟着物理走
· odom→base_footprint TF = [0.848, 0, 0]，且只有这一个来源
· 全量 colcon test：130 tests, 0 failures, 0 errors（含 nav2 + mock 端到端）

文档同步：robot-flows.md（6.1/6.2/7.2/9 四处表与说明）、file-map.md（桥的方向表）、
mock-robot-node.md、robot_sdk_gazebo/README.md 里"底盘由 gz DiffDrive 驱动""桥 9 条"
"cmd_vel 是 Twist"的口径全部改准。

File: src/robot_description/urdf/mobile_manipulator.urdf.xacro (robot description, xacro)
@@ -464,19 +464,8 @@
   </xacro:macro>
   <gazebo>
-    <plugin filename="gz-sim-diff-drive-system" name="gz::sim::systems::DiffDrive">
-      <left_joint>left_wheel_joint</left_joint>
-      <right_joint>right_wheel_joint</right_joint>
-      <wheel_separation>${2.0 * wheel_offset_y}</wheel_separation>
-      <wheel_radius>${wheel_radius}</wheel_radius>
-      <max_linear_acceleration>1.0</max_linear_acceleration>
-      <min_linear_acceleration>-1.0</min_linear_acceleration>
-      <max_angular_acceleration>2.0</max_angular_acceleration>
-      <min_angular_acceleration>-2.0</min_angular_acceleration>
-      <topic>/cmd_vel</topic>
-      <odom_topic>/odom</odom_topic>
-      <frame_id>odom</frame_id>
-      <child_frame_id>base_footprint</child_frame_id>
-      <odom_publish_frequency>50</odom_publish_frequency>
-    </plugin>
+    <!-- 底盘**不再**用 gz 私有的 DiffDrive 插件：车轮已纳入 ros2_control（见文件末的
+         <ros2_control>），由标准控制器 diff_drive_controller 驱动，/odom 也由它发。
+         ⇒ 底盘与手臂走**同一套**驱动机制；接真机时换的是同一个硬件插件（只换 plugin 名）。
+         ⚠️ 留着的代价是：gz DiffDrive 会和 ros2_control 抢同一个关节，并且产生**两个** /odom 源。 -->
     <!-- ⚠️ gazebo 模式下手臂的关节状态由 ros2_control 的 broadcaster 发，这里**只补车轮** ——
          少了它们 MoveIt 的当前状态永远不完整（一直 warn "complete state ... not yet known"）。
@@ -598,7 +587,11 @@
   </xacro:if>
   <!-- ============================ ros2_control ============================= -->
-  <!-- 给 ros2_control 用的：声明关节、接口、硬件插件，只声明要控的 7 个（车轮没人控）。
+  <!-- 给 ros2_control 用的：声明关节、接口、硬件插件。手臂 7 个 + 车轮 2 个。
+       ⚠️ 车轮用**速度**接口（差速底盘本来就是速度控制），手臂用位置接口。
        ⚠️ 插件由 `hardware` 参数二选一 —— 默认 mock（假硬件，命令即状态，不需要 Gazebo）；
-       gazebo 模式换成 gz_ros2_control，那时 MoveIt 才能**真的**驱动仿真里的机器人。 -->
+       gazebo 模式换成 gz_ros2_control，那时 MoveIt 才能**真的**驱动仿真里的机器人，
+       车轮也才由 diff_drive_controller 驱动（见 config/ros2_control.yaml）。
+       ⚠️ 车轮的 /joint_states 仍由 gz 的 JointStatePublisher 经桥发出（下面 <gazebo> 里），
+          所以 `joint_state_broadcaster` 只列手臂 —— 否则同一个关节会有两个发布者。 -->
   <ros2_control name="mobile_manipulator" type="system">
     <hardware>
@@ -638,4 +631,15 @@
       <state_interface name="position"/>
     </joint>
+    <!-- 车轮：差速底盘用速度接口；状态给 position（里程计要积分它）+ velocity。 -->
+    <joint name="left_wheel_joint">
+      <command_interface name="velocity"/>
+      <state_interface name="position"/>
+      <state_interface name="velocity"/>
+    </joint>
+    <joint name="right_wheel_joint">
+      <command_interface name="velocity"/>
+      <state_interface name="position"/>
+      <state_interface name="velocity"/>
+    </joint>
   </ros2_control>
 </robot>
